Commit message: Added explanation to run it with another package
If you want to run this package on <url type="repository">https://github.com/start-jsk/denso</url>  just change the following

denso_description/meshes/denso

with 

vs060/model/meshes

File: vs060_gazebo/urdf/vs060-gazebo.xacro (robot description, xacro)
@@ -17,5 +17,5 @@
       <origin xyz="0 0 0" rpy="0 -0 0"/>
       <geometry>
-        <mesh filename="package://vs060/model/meshes/BASE_mesh.stl"/>
+        <mesh filename="package://denso_description/meshes/denso/BASE_mesh.stl"/>
       </geometry>
     </visual>
@@ -23,5 +23,5 @@
       <origin xyz="0 0 0" rpy="0 -0 0"/>
       <geometry>
-        <mesh filename="package://vs060/model/meshes/BASE_mesh.stl"/>
+        <mesh filename="package://denso_description/meshes/denso/BASE_mesh.stl"/>
       </geometry>
     </collision>
@@ -36,5 +36,5 @@
       <origin xyz="0 4.04121e-17 0.182" rpy="0 -0 0"/>
       <geometry>
-        <mesh filename="package://vs060/model/meshes/J1_mesh.stl"/>
+        <mesh filename="package://denso_description/meshes/denso/J1_mesh.stl"/>
       </geometry>
     </visual>
@@ -42,5 +42,5 @@
       <origin xyz="0 4.04121e-17 0.182" rpy="0 -0 0"/>
       <geometry>
-        <mesh filename="package://vs060/model/meshes/J1_mesh.stl"/>
+        <mesh filename="package://denso_description/meshes/denso/J1_mesh.stl"/>
       </geometry>
     </collision>
@@ -55,5 +55,5 @@
       <origin xyz="0 3.61933e-17 0.163" rpy="0 -0 0"/>
       <geometry>
-        <mesh filename="package://vs060/model/meshes/J2_mesh.stl"/>
+        <mesh filename="package://denso_description/meshes/denso/J2_mesh.stl"/>
       </geometry>
     </visual>
@@ -61,5 +61,5 @@
       <origin xyz="0 3.61933e-17 0.163" rpy="0 -0 0"/>
       <geometry>
-        <mesh filename="package://vs060/model/meshes/J2_mesh.stl"/>
+        <mesh filename="package://denso_description/meshes/denso/J2_mesh.stl"/>
       </geometry>
     </collision>
@@ -74,5 +74,5 @@
       <origin xyz="0 6.77236e-17 0.305" rpy="0 -0 0"/>
       <geometry>
-        <mesh filename="package://vs060/model/meshes/J3_mesh.stl"/>
+        <mesh filename="package://denso_description/meshes/denso/J3_mesh.stl"/>
       </geometry>
     </visual>
@@ -80,5 +80,5 @@
       <origin xyz="0 6.77236e-17 0.305" rpy="0 -0 0"/>
       <geometry>
-        <mesh filename="package://vs060/model/meshes/J3_mesh.stl"/>
+        <mesh filename="package://denso_description/meshes/denso/J3_mesh.stl"/>
       </geometry>
     </collision>
@@ -93,5 +93,5 @@
       <origin xyz="-0.01 3.66374e-17 0.165" rpy="0 -0 0"/>
       <geometry>
-        <mesh filename="package://vs060/model/meshes/J4_mesh.stl"/>
+        <mesh filename="package://denso_description/meshes/denso/J4_mesh.stl"/>
       </geometry>
     </visual>
@@ -99,5 +99,5 @@
       <origin xyz="-0.01 3.66374e-17 0.165" rpy="0 -0 0"/>
       <geometry>
-        <mesh filename="package://vs060/model/meshes/J4_mesh.stl"/>
+        <mesh filename="package://denso_description/meshes/denso/J4_mesh.stl"/>
       </geometry>
     </collision>
@@ -112,5 +112,5 @@
       <origin xyz="0 2.9976e-17 0.135" rpy="0 -0 0"/>
       <geometry>
-        <mesh filename="package://vs060/model/meshes/J5_mesh.stl"/>
+        <mesh filename="package://denso_description/meshes/denso/J5_mesh.stl"/>
       </geometry>
     </visual>
@@ -118,5 +118,5 @@
       <origin xyz="0 2.9976e-17 0.135" rpy="0 -0 0"/>
       <geometry>
-        <mesh filename="package://vs060/model/meshes/J5_mesh.stl"/>
+        <mesh filename="package://denso_description/meshes/denso/J5_mesh.stl"/>
       </geometry>
     </collision>
@@ -131,5 +131,5 @@
       <origin xyz="0 1.55431e-17 0.07" rpy="0 -0 0"/>
       <geometry>
-        <mesh filename="package://vs060/model/meshes/Flange_mesh.stl"/>
+        <mesh filename="package://denso_description/meshes/denso/Flange_mesh.stl"/>
       </geometry>
     </visual>
@@ -137,5 +137,5 @@
       <origin xyz="0 1.55431e-17 0.07" rpy="0 -0 0"/>
       <geometry>
-        <mesh filename="package://vs060/model/meshes/Flange_mesh.stl"/>
+        <mesh filename="package://denso_description/meshes/denso/Flange_mesh.stl"/>
       </geometry>
     </collision>
